Commit message: add maddpg and env

File: src/turtlebot3/turtlebot3_description/urdf/turtlebot3_burger.gazebo.xacro (robot description, xacro)
@@ -5,4 +5,9 @@
   <!-- Add robot namespace as a property -->
   <xacro:property name="robot_namespace" value="$(arg robot_namespace)"/>
+  <!--
+  <xacro:property name="robot_x" value="$(arg robot_x)"/>
+  <xacro:property name="robot_y" value="$(arg robot_y)"/>
+  <xacro:property name="robot_yaw" value="$(arg robot_yaw)"/>
+  -->
   <gazebo reference="base_link">
     <material>Gazebo/DarkGrey</material>
@@ -65,4 +70,8 @@
       <odometryRate>10.0</odometryRate>
       <isGroundTruth>false</isGroundTruth>
+      <odometrySource>world</odometrySource>
+      <!--
+      <initialPose>$(arg robot_x) $(arg robot_y) 0 $(arg robot_yaw) 0 0</initialPose>
+      -->
       <alwaysOn>true</alwaysOn>
     </plugin>

File: src/turtlebot3/turtlebot3_description/urdf/turtlebot3_burger.urdf.xacro (robot description, xacro)
@@ -4,13 +4,13 @@
   <xacro:property name="robot_namespace" value="$(arg robot_namespace)"/>
   <xacro:include filename="$(find turtlebot3_description)/urdf/common_properties.xacro"/>
-  <xacro:include filename="$(find turtlebot3_description)/urdf/turtlebot3_burger.gazebo.xacro"/>
-  <!-- Add odom as a fixed link
-  <link name="odom"/>
-  <joint name="odom_joint" type="fixed">
-    <parent link="odom"/>
-    <child link="base_footprint"/>
-    <origin xyz="0 0 0" rpy="0 0 0"/>
-  </joint>
-  -->
+  <!-- 包含子文件并传递参数 -->
+  <xacro:include filename="$(find turtlebot3_description)/urdf/turtlebot3_burger.gazebo.xacro">
+      <xacro:arg name="robot_namespace" value="$(arg robot_namespace)"/>
+      <!--
+      <xacro:arg name="robot_x" value="$(arg robot_x)"/>
+      <xacro:arg name="robot_y" value="$(arg robot_y)"/>
+      <xacro:arg name="robot_yaw" value="$(arg robot_yaw)"/>
+      -->
+  </xacro:include>
   <link name="base_footprint"/>
   <joint name="base_joint" type="fixed">
